File: ai03-pcb-guide.sch (KiCad schematic (older format))
At the start: 34 parts, among them J1 USB_mini_micro_B, SW1 SW_Push, U1 ATmega32U4-AU, Y1 Crystal_GND24_Small

Commit message: using pro micro instead,added tht diodes,firmware
Parts:
- removed C1, C2, C5: 0.1uF, Capacitors_SMD:C_0805, symbol ai03-pcb-guide-rescue:C_Small-Device
- removed C3, C4: 22pF, Capacitors_SMD:C_0805, symbol ai03-pcb-guide-rescue:C_Small-Device
- removed C6: 1uF, Capacitors_SMD:C_0805, symbol ai03-pcb-guide-rescue:C_Small-Device
- removed C7: 10uF, Capacitors_SMD:C_0805, symbol ai03-pcb-guide-rescue:C_Small-Device
- removed F1: 500mA, Fuse:Fuse_1206_3216Metric, symbol ai03-pcb-guide-rescue:Polyfuse_Small-Device
- removed J1: USB_mini_micro_B, keyboard_parts:USB_microB, symbol keyboard_parts:USB_mini_micro_B
- removed R1, R2: 22, Resistors_SMD:R_0805, symbol ai03-pcb-guide-rescue:R_Small-Device
- removed R3, R4: 10k, Resistors_SMD:R_0805, symbol ai03-pcb-guide-rescue:R_Small-Device
- removed SW1: SW_Push, random-keyboard-parts:SKQG-1155865, symbol ai03-pcb-guide-rescue:SW_Push-Switch
- removed U1: ATmega32U4-AU, Housings_QFP:TQFP-44_10x10mm_Pitch0.8mm, symbol ai03-pcb-guide-rescue:ATmega32U4-AU-MCU_Microchip_ATmega
- removed Y1: Crystal_GND24_Small, Crystals:Crystal_SMD_3225-4pin_3.2x2.5mm, symbol ai03-pcb-guide-rescue:Crystal_GND24_Small-Device
- added U1: ProMicro, promicro:ProMicro, symbol promicro:ProMicro
- D1, D2, D3, D4, D5, D6, D7, D8, D9: footprint Diode_SMD:D_SOD-123 -> Diode_THT:D_DO-15_P5.08mm_Vertical_AnodeUp
Connections:
- net COL0: now also U1.16 (B1)
- net COL1: now also U1.15 (B3)
- net COL2: now also U1.14 (B2)
- net ROW0: now also U1.20 (F4)
- net ROW1: now also U1.19 (F5)
- net ROW2: now also U1.18 (F6)
